Commit message: panda,robotiq urdf seperated

File: icra19/description/panda_robotiq.urdf.xacro (robot description, xacro)
@@ -1,12 +1,7 @@
 <?xml version="1.0" encoding="utf-8"?>
 <robot xmlns:xacro="http://www.ros.org/wiki/xacro" name="panda_robotiq">
-  <xacro:include filename="$(find franka_description)/robots/panda_arm.xacro"/>
+  <xacro:include filename="$(find icra19)/description/panda_robotiq_connector_macro.xacro"/>
   <xacro:include filename="$(find robotiq_2f_c2_gripper_visualization)/urdf/robotiq_c2_model_macro.xacro"/>
-  <xacro:panda_arm/>
-  <joint name="panda_robotiq_attachment_joint" type="fixed">
-    <origin xyz="0 0 0" rpy="0 -1.5707963268 0"/>
-    <parent link="panda_link8"/>
-    <child link="robotiq_85_adapter_link"/>
-  </joint>
+  <xacro:panda_robotiq_connector/>
   <xacro:robotiq_c2_model prefix=""/>
 </robot>

Commit message: switched to Danfoa's robotiq repository

File: icra19/description/panda_robotiq.urdf.xacro (robot description, xacro)
@@ -2,6 +2,8 @@
 <robot xmlns:xacro="http://www.ros.org/wiki/xacro" name="panda_robotiq">
   <xacro:include filename="$(find icra19)/description/panda_robotiq_connector_macro.xacro"/>
-  <xacro:include filename="$(find robotiq_2f_c2_gripper_visualization)/urdf/robotiq_c2_model_macro.xacro"/>
+  <xacro:include filename="$(find robotiq_2f_85_gripper_visualization)/urdf/robotiq_arg2f_85_model.xacro"/>
   <xacro:panda_robotiq_connector/>
-  <xacro:robotiq_c2_model prefix=""/>
+  <!--
+  <xacro:robotiq_arg2f_85_model prefix=""/>
+  -->
 </robot>

File: icra19/description/panda_robotiq_connector_macro.xacro (robot description, xacro)
@@ -4,7 +4,7 @@
     <link name="panda_link8"/>
     <joint name="panda_robotiq_attachment_joint" type="fixed">
-      <origin xyz="0 0 0" rpy="0 -1.5707963268 0"/>
+      <origin xyz="0 0 0" rpy="0 0 0"/>
       <parent link="panda_link8"/>
-      <child link="robotiq_85_adapter_link"/>
+      <child link="robotiq_arg2f_base_link"/>
     </joint>
   </xacro:macro>

Commit message: working on publishable version

File: icra19/description/panda_robotiq.urdf.xacro (robot description, xacro)
@@ -1,9 +1,6 @@
 <?xml version="1.0" encoding="utf-8"?>
 <robot xmlns:xacro="http://www.ros.org/wiki/xacro" name="panda_robotiq">
-  <xacro:include filename="$(find icra19)/description/panda_robotiq_connector_macro.xacro"/>
+  <xacro:include filename="$(find icra19)/description/panda_robotiq_connector_joint.xacro"/>
   <xacro:include filename="$(find robotiq_2f_85_gripper_visualization)/urdf/robotiq_arg2f_85_model.xacro"/>
   <xacro:panda_robotiq_connector/>
-  <!--
-  <xacro:robotiq_arg2f_85_model prefix=""/>
-  -->
 </robot>

File: icra19/description/panda_robotiq_connector_joint.xacro (robot description, xacro)
@@ -4,5 +4,5 @@
     <link name="panda_link8"/>
     <joint name="panda_robotiq_attachment_joint" type="fixed">
-      <origin xyz="0 0 0" rpy="0 0 0"/>
+      <origin xyz="0 0 0" rpy="0 0 1.5707963268"/>
       <parent link="panda_link8"/>
       <child link="robotiq_arg2f_base_link"/>
